File: hardware/bq76920/AFE.sch (KiCad schematic (older format))
At the start: 27 parts, among them Q1 PSMN2R6-40YS, Q2 SI2337DS-T1-E3, Q3 PSMN2R6-40YS, U1 bq76920

Commit message: clean up, adnotate, footprints
Signed-off-by: Ene Alexandru <ene.alexandru@gmail.com>
Parts:
- C5, C7, C8: footprint Capacitor_SMD:C_1210_3225Metric_Pad1.42x2.65mm_HandSolder -> Capacitor_SMD:C_1206_3216Metric_Pad1.42x1.75mm_HandSolder
Changed lines of the file:
@@
 F 0 "C5" H 4858 1054 50  0000 R CNN
 F 1 "C1206C475K5RACTU" H 4858 1145 50  0000 R CNN
-F 2 "Capacitor_SMD:C_1210_3225Metric_Pad1.42x2.65mm_HandSolder" H 4950 1100 50  0001 C CNN
+F 2 "Capacitor_SMD:C_1206_3216Metric_Pad1.42x1.75mm_HandSolder" H 4950 1100 50  0001 C CNN
 F 3 "~" H 4950 1100 50  0001 C CNN
 	1    4950 1100
@@
 F 0 "C7" H 5908 1954 50  0000 R CNN
 F 1 "C1206C475K5RACTU" H 5950 2100 50  0000 R CNN
-F 2 "Capacitor_SMD:C_1210_3225Metric_Pad1.42x2.65mm_HandSolder" H 6000 2000 50  0001 C CNN
+F 2 "Capacitor_SMD:C_1206_3216Metric_Pad1.42x1.75mm_HandSolder" H 6000 2000 50  0001 C CNN
 F 3 "~" H 6000 2000 50  0001 C CNN
 	1    6000 2000
@@
 F 0 "C8" H 8458 1954 50  0000 R CNN
 F 1 "C1206C475K5RACTU" H 8458 2045 50  0000 R CNN
-F 2 "Capacitor_SMD:C_1210_3225Metric_Pad1.42x2.65mm_HandSolder" H 8550 2000 50  0001 C CNN
+F 2 "Capacitor_SMD:C_1206_3216Metric_Pad1.42x1.75mm_HandSolder" H 8550 2000 50  0001 C CNN
 F 3 "~" H 8550 2000 50  0001 C CNN
 	1    8550 2000
