File: hardware/bq76920/bq76920.sch (KiCad schematic (older format))
At the start: 10 parts, among them J1 BAT+, J2 Conn_01x06, J3 therm, J4 boot_switch, J5 BAT-, J6 PACK+, J7 PACK-

Commit message: clean up, adnotate, footprints
Signed-off-by: Ene Alexandru <ene.alexandru@gmail.com>
Parts:
- J8: renamed from J?; footprint (none) -> Connector_PinHeader_2.54mm:PinHeader_1x04_P2.54mm_Vertical
Changed lines of the file:
@@
 	5100 2200 6200 2200
 $Comp
-L Connector_Generic:Conn_01x04 J?
+L Connector_Generic:Conn_01x04 J8
 U 1 1 5E14DD4B
 P 10150 2000
-F 0 "J?" H 10230 1992 50  0000 L CNN
+F 0 "J8" H 10230 1992 50  0000 L CNN
 F 1 "Conn_01x04" H 10230 1901 50  0000 L CNN
-F 2 "" H 10150 2000 50  0001 C CNN
+F 2 "Connector_PinHeader_2.54mm:PinHeader_1x04_P2.54mm_Vertical" H 10150 2000 50  0001 C CNN
 F 3 "~" H 10150 2000 50  0001 C CNN
 	1    10150 2000

Commit message: final pcb version
Signed-off-by: Ene Alexandru <ene.alexandru@gmail.com>
Connections:
- net bq76920 section/RAW_PACK- is gone; now on net BAT+: J6.1 (Pin_1)
Changed lines of the file:
@@
 F14 "BAT_THERM" I L 4000 2300 50
 F15 "REGOUT" I R 5100 1900 50
-F16 "RAW_PACK-" I R 5100 1600 50
-F17 "PACK-" I R 5100 2750 50
+F16 "PACK-" I R 5100 2750 50
 $EndSheet
 $Sheet
@@
 	3150 2750 3150 4350
 Wire Wire Line
-	5100 1600 6050 1600
-Wire Wire Line
-	6050 1600 6050 900
-Wire Wire Line
-	6050 900  9950 900
-Wire Wire Line
 	5100 2750 6050 2750
 Wire Wire Line
@@
 Wire Wire Line
 	5100 2200 6200 2200
+Wire Wire Line
+	9950 1900 7350 1900
+Wire Wire Line
+	7350 2000 9950 2000
+Wire Wire Line
+	9950 2100 7350 2100
+Wire Wire Line
+	7350 2200 9950 2200
+Wire Wire Line
+	3050 900  9950 900
+Connection ~ 3050 900
 $Comp
 L Connector_Generic:Conn_01x04 J8
@@
 	1    0    0    -1
 $EndComp
-Wire Wire Line
-	9950 1900 7350 1900
-Wire Wire Line
-	7350 2000 9950 2000
-Wire Wire Line
-	9950 2100 7350 2100
-Wire Wire Line
-	7350 2200 9950 2200
 $EndSCHEMATC
