File: hardware/bq76920/cpu.sch (KiCad schematic (older format))
At the start: 17 parts

Commit message: clean up, adnotate, footprints
Signed-off-by: Ene Alexandru <ene.alexandru@gmail.com>
Parts:
- C16, C17, C18, C19, C9: renamed from C?; footprint (none) -> Capacitor_SMD:C_0805_2012Metric_Pad1.15x1.40mm_HandSolder
- D11, D12, D13: renamed from D?; footprint (none) -> Capacitor_SMD:C_1206_3216Metric_Pad1.42x1.75mm_HandSolder
- J10: renamed from J?; footprint (none) -> Connector_PinHeader_2.54mm:PinHeader_1x02_P2.54mm_Vertical
- J9: renamed from J?; footprint (none) -> Connector_PinHeader_2.54mm:PinHeader_1x05_P2.54mm_Vertical
- R32, R33, R34, R35, R36: renamed from R?; footprint (none) -> Resistor_SMD:R_0815_2038Metric_Pad1.53x4.00mm_HandSolder
- U2: renamed from U?; footprint (none) -> Package_SO:SOIC-8_3.9x4.9mm_P1.27mm
- gave numbers to parts that had none: 1
Changed lines of the file:
@@
 PACK_SDA
 $Comp
-L MCU_ST_STM32L0:STM32L031F4Px U?
+L MCU_ST_STM32L0:STM32L031F4Px U3
 U 1 1 5E142A54
 P 4950 3850
-F 0 "U?" H 4600 4550 50  0000 C CNN
+F 0 "U3" H 4600 4550 50  0000 C CNN
 F 1 "STM32L031F4Px" H 5350 3050 50  0000 C CNN
 F 2 "Package_SO:TSSOP-20_4.4x6.5mm_P0.65mm" H 4550 3150 50  0001 R CNN
@@
 $EndComp
 $Comp
-L Connector_Generic:Conn_01x05 J?
+L Connector_Generic:Conn_01x05 J9
 U 1 1 5E133C66
 P 1350 6550
-F 0 "J?" H 1270 6967 50  0000 C CNN
+F 0 "J9" H 1270 6967 50  0000 C CNN
 F 1 "Conn_01x05" H 1270 6876 50  0000 C CNN
-F 2 "" H 1350 6550 50  0001 C CNN
+F 2 "Connector_PinHeader_2.54mm:PinHeader_1x05_P2.54mm_Vertical" H 1350 6550 50  0001 C CNN
 F 3 "~" H 1350 6550 50  0001 C CNN
 	1    1350 6550
@@
 $EndComp
 $Comp
-L Device:R_Small R?
+L Device:R_Small R33
 U 1 1 5E133DEA
 P 2700 6200
-F 0 "R?" H 2759 6246 50  0000 L CNN
+F 0 "R33" H 2759 6246 50  0000 L CNN
 F 1 "10k" H 2759 6155 50  0000 L CNN
-F 2 "" H 2700 6200 50  0001 C CNN
+F 2 "Resistor_SMD:R_0815_2038Metric_Pad1.53x4.00mm_HandSolder" H 2700 6200 50  0001 C CNN
 F 3 "~" H 2700 6200 50  0001 C CNN
 	1    2700 6200
@@
 	2700 6350 2700 6300
 $Comp
-L power:+3V3 #PWR?
+L power:+3V3 #PWR0101
 U 1 1 5E133EE0
 P 1350 1200
-F 0 "#PWR?" H 1350 1050 50  0001 C CNN
+F 0 "#PWR0101" H 1350 1050 50  0001 C CNN
 F 1 "+3V3" H 1365 1373 50  0000 C CNN
 F 2 "" H 1350 1200 50  0001 C CNN
@@
 	1350 1300 1200 1300
 $Comp
-L power:+3V3 #PWR?
+L power:+3V3 #PWR0102
 U 1 1 5E133F22
 P 2700 6000
-F 0 "#PWR?" H 2700 5850 50  0001 C CNN
+F 0 "#PWR0102" H 2700 5850 50  0001 C CNN
 F 1 "+3V3" H 2715 6173 50  0000 C CNN
 F 2 "" H 2700 6000 50  0001 C CNN
@@
 $EndComp
 $Comp
-L Device:C_Small C?
+L Device:C_Small C18
 U 1 1 5E134013
 P 2700 6500
-F 0 "C?" H 2792 6546 50  0000 L CNN
+F 0 "C18" H 2792 6546 50  0000 L CNN
 F 1 "1n" H 2792 6455 50  0000 L CNN
-F 2 "" H 2700 6500 50  0001 C CNN
+F 2 "Capacitor_SMD:C_0805_2012Metric_Pad1.15x1.40mm_HandSolder" H 2700 6500 50  0001 C CNN
 F 3 "~" H 2700 6500 50  0001 C CNN
 	1    2700 6500
@@
 $EndComp
 $Comp
-L power:GND #PWR?
+L power:GND #PWR0103
 U 1 1 5E1340FD
 P 2700 6700
-F 0 "#PWR?" H 2700 6450 50  0001 C CNN
+F 0 "#PWR0103" H 2700 6450 50  0001 C CNN
 F 1 "GND" H 2705 6527 50  0000 C CNN
 F 2 "" H 2700 6700 50  0001 C CNN
@@
 	2700 6700 2700 6600
 $Comp
-L Device:R_Small R?
+L Device:R_Small R32
 U 1 1 5E134235
 P 1600 6950
-F 0 "R?" H 1659 6996 50  0000 L CNN
+F 0 "R32" H 1659 6996 50  0000 L CNN
 F 1 "10k" H 1659 6905 50  0000 L CNN
-F 2 "" H 1600 6950 50  0001 C CNN
+F 2 "Resistor_SMD:R_0815_2038Metric_Pad1.53x4.00mm_HandSolder" H 1600 6950 50  0001 C CNN
 F 3 "~" H 1600 6950 50  0001 C CNN
 	1    1600 6950
@@
 	2700 6000 2700 6100
 $Comp
-L power:GND #PWR?
+L power:GND #PWR0104
 U 1 1 5E134F0A
 P 1600 7150
-F 0 "#PWR?" H 1600 6900 50  0001 C CNN
+F 0 "#PWR0104" H 1600 6900 50  0001 C CNN
 F 1 "GND" H 1605 6977 50  0000 C CNN
 F 2 "" H 1600 7150 50  0001 C CNN
@@
 	1600 6750 1700 6750
 $Comp
-L power:GND #PWR?
+L power:GND #PWR0105
 U 1 1 5E13539F
 P 2100 7150
-F 0 "#PWR?" H 2100 6900 50  0001 C CNN
+F 0 "#PWR0105" H 2100 6900 50  0001 C CNN
 F 1 "GND" H 2105 6977 50  0000 C CNN
 F 2 "" H 2100 7150 50  0001 C CNN
@@
 SWCLK
 $Comp
-L power:+3V3 #PWR?
+L power:+3V3 #PWR0106
 U 1 1 5E1371AD
 P 4950 3050
-F 0 "#PWR?" H 4950 2900 50  0001 C CNN
+F 0 "#PWR0106" H 4950 2900 50  0001 C CNN
 F 1 "+3V3" H 4965 3223 50  0000 C CNN
 F 2 "" H 4950 3050 50  0001 C CNN
@@
 	4950 3100 4950 3150
 $Comp
-L power:GND #PWR?
+L power:GND #PWR0107
 U 1 1 5E13770A
 P 4950 4750
-F 0 "#PWR?" H 4950 4500 50  0001 C CNN
+F 0 "#PWR0107" H 4950 4500 50  0001 C CNN
 F 1 "GND" H 4955 4577 50  0000 C CNN
 F 2 "" H 4950 4750 50  0001 C CNN
@@
 P 3900 1250
 AR Path="/5E13BDED" Ref="U?"  Part="1"
-AR Path="/5E142913/5E13BDED" Ref="U?"  Part="1"
-F 0 "U?" H 4225 1515 50  0000 C CNN
+AR Path="/5E142913/5E13BDED" Ref="U2"  Part="1"
+F 0 "U2" H 4225 1515 50  0000 C CNN
 F 1 "ISO7021" H 4225 1424 50  0000 C CNN
-F 2 "" H 3900 1250 50  0001 C CNN
+F 2 "Package_SO:SOIC-8_3.9x4.9mm_P1.27mm" H 3900 1250 50  0001 C CNN
 F 3 "" H 3900 1250 50  0001 C CNN
 	1    3900 1250
@@
 $EndComp
 $Comp
-L power:GND #PWR?
+L power:GND #PWR0108
 U 1 1 5E13BED3
 P 3750 1600
-F 0 "#PWR?" H 3750 1350 50  0001 C CNN
+F 0 "#PWR0108" H 3750 1350 50  0001 C CNN
 F 1 "GND" H 3755 1427 50  0000 C CNN
 F 2 "" H 3750 1600 50  0001 C CNN
@@
 	3750 1600 3750 1550
 $Comp
-L power:+3V3 #PWR?
+L power:+3V3 #PWR0109
 U 1 1 5E13D8E9
 P 3750 1200
-F 0 "#PWR?" H 3750 1050 50  0001 C CNN
+F 0 "#PWR0109" H 3750 1050 50  0001 C CNN
 F 1 "+3V3" H 3765 1373 50  0000 C CNN
 F 2 "" H 3750 1200 50  0001 C CNN
@@
 	3750 1250 3800 1250
 $Comp
-L Device:C_Small C?
+L Device:C_Small C9
 U 1 1 5E13DDCE
 P 1350 1450
-F 0 "C?" H 1442 1496 50  0000 L CNN
+F 0 "C9" H 1442 1496 50  0000 L CNN
 F 1 "100nF" H 1442 1405 50  0000 L CNN
-F 2 "" H 1350 1450 50  0001 C CNN
+F 2 "Capacitor_SMD:C_0805_2012Metric_Pad1.15x1.40mm_HandSolder" H 1350 1450 50  0001 C CNN
 F 3 "~" H 1350 1450 50  0001 C CNN
 	1    1350 1450
@@
 $EndComp
 $Comp
-L Device:C_Small C?
+L Device:C_Small C16
 U 1 1 5E13DE7D
 P 1800 1450
-F 0 "C?" H 1892 1496 50  0000 L CNN
+F 0 "C16" H 1892 1496 50  0000 L CNN
 F 1 "100nF" H 1892 1405 50  0000 L CNN
-F 2 "" H 1800 1450 50  0001 C CNN
+F 2 "Capacitor_SMD:C_0805_2012Metric_Pad1.15x1.40mm_HandSolder" H 1800 1450 50  0001 C CNN
 F 3 "~" H 1800 1450 50  0001 C CNN
 	1    1800 1450
@@
 $EndComp
 $Comp
-L Device:C_Small C?
+L Device:C_Small C17
 U 1 1 5E13DFFD
 P 2250 1450
-F 0 "C?" H 2342 1496 50  0000 L CNN
+F 0 "C17" H 2342 1496 50  0000 L CNN
 F 1 "100nF" H 2342 1405 50  0000 L CNN
-F 2 "" H 2250 1450 50  0001 C CNN
+F 2 "Capacitor_SMD:C_0805_2012Metric_Pad1.15x1.40mm_HandSolder" H 2250 1450 50  0001 C CNN
 F 3 "~" H 2250 1450 50  0001 C CNN
 	1    2250 1450
@@
 $EndComp
 $Comp
-L power:GND #PWR?
+L power:GND #PWR0110
 U 1 1 5E13E117
 P 1350 1650
-F 0 "#PWR?" H 1350 1400 50  0001 C CNN
+F 0 "#PWR0110" H 1350 1400 50  0001 C CNN
 F 1 "GND" H 1355 1477 50  0000 C CNN
 F 2 "" H 1350 1650 50  0001 C CNN
@@
 Connection ~ 1800 1600
 $Comp
-L Device:C_Small C?
+L Device:C_Small C19
 U 1 1 5E140D1B
 P 5250 1400
-F 0 "C?" H 5342 1446 50  0000 L CNN
+F 0 "C19" H 5342 1446 50  0000 L CNN
 F 1 "100nF" H 5342 1355 50  0000 L CNN
-F 2 "" H 5250 1400 50  0001 C CNN
+F 2 "Capacitor_SMD:C_0805_2012Metric_Pad1.15x1.40mm_HandSolder" H 5250 1400 50  0001 C CNN
 F 3 "~" H 5250 1400 50  0001 C CNN
 	1    5250 1400
@@
 $EndComp
 $Comp
-L Connector_Generic:Conn_01x02 J?
+L Connector_Generic:Conn_01x02 J10
 U 1 1 5E140FA3
 P 6400 3550
-F 0 "J?" H 6480 3542 50  0000 L CNN
+F 0 "J10" H 6480 3542 50  0000 L CNN
 F 1 "Conn_01x02" H 6480 3451 50  0000 L CNN
-F 2 "" H 6400 3550 50  0001 C CNN
+F 2 "Connector_PinHeader_2.54mm:PinHeader_1x02_P2.54mm_Vertical" H 6400 3550 50  0001 C CNN
 F 3 "~" H 6400 3550 50  0001 C CNN
 	1    6400 3550
@@
 Connection ~ 5250 1550
 $Comp
-L Device:LED_Small D?
+L Device:LED_Small D11
 U 1 1 5E153362
 P 6500 4550
-F 0 "D?" V 6546 4482 50  0000 R CNN
+F 0 "D11" V 6546 4482 50  0000 R CNN
 F 1 "APTD3216SURCK" V 6455 4482 50  0000 R CNN
-F 2 "" V 6500 4550 50  0001 C CNN
+F 2 "Capacitor_SMD:C_1206_3216Metric_Pad1.42x1.75mm_HandSolder" V 6500 4550 50  0001 C CNN
 F 3 "~" V 6500 4550 50  0001 C CNN
 	1    6500 4550
@@
 $EndComp
 $Comp
-L Device:R_Small R?
+L Device:R_Small R34
 U 1 1 5E155044
 P 6500 4250
-F 0 "R?" H 6559 4296 50  0000 L CNN
+F 0 "R34" H 6559 4296 50  0000 L CNN
 F 1 "10k" H 6559 4205 50  0000 L CNN
-F 2 "" H 6500 4250 50  0001 C CNN
+F 2 "Resistor_SMD:R_0815_2038Metric_Pad1.53x4.00mm_HandSolder" H 6500 4250 50  0001 C CNN
 F 3 "~" H 6500 4250 50  0001 C CNN
 	1    6500 4250
@@
 $EndComp
 $Comp
-L Device:LED_Small D?
+L Device:LED_Small D12
 U 1 1 5E15CED0
 P 7400 4550
-F 0 "D?" V 7446 4482 50  0000 R CNN
+F 0 "D12" V 7446 4482 50  0000 R CNN
 F 1 "APTD3216SURCK" V 7355 4482 50  0000 R CNN
-F 2 "" V 7400 4550 50  0001 C CNN
+F 2 "Capacitor_SMD:C_1206_3216Metric_Pad1.42x1.75mm_HandSolder" V 7400 4550 50  0001 C CNN
 F 3 "~" V 7400 4550 50  0001 C CNN
 	1    7400 4550
@@
 $EndComp
 $Comp
-L Device:R_Small R?
+L Device:R_Small R35
 U 1 1 5E15CEDA
 P 7400 4250
-F 0 "R?" H 7459 4296 50  0000 L CNN
+F 0 "R35" H 7459 4296 50  0000 L CNN
 F 1 "10k" H 7459 4205 50  0000 L CNN
-F 2 "" H 7400 4250 50  0001 C CNN
+F 2 "Resistor_SMD:R_0815_2038Metric_Pad1.53x4.00mm_HandSolder" H 7400 4250 50  0001 C CNN
 F 3 "~" H 7400 4250 50  0001 C CNN
 	1    7400 4250
@@
 $EndComp
 $Comp
-L Device:LED_Small D?
+L Device:LED_Small D13
 U 1 1 5E16427F
 P 8250 4550
-F 0 "D?" V 8296 4482 50  0000 R CNN
+F 0 "D13" V 8296 4482 50  0000 R CNN
 F 1 "APTD3216SURCK" V 8205 4482 50  0000 R CNN
-F 2 "" V 8250 4550 50  0001 C CNN
+F 2 "Capacitor_SMD:C_1206_3216Metric_Pad1.42x1.75mm_HandSolder" V 8250 4550 50  0001 C CNN
 F 3 "~" V 8250 4550 50  0001 C CNN
 	1    8250 4550
@@
 $EndComp
 $Comp
-L Device:R_Small R?
+L Device:R_Small R36
 U 1 1 5E164693
 P 8250 4250
-F 0 "R?" H 8309 4296 50  0000 L CNN
+F 0 "R36" H 8309 4296 50  0000 L CNN
 F 1 "10k" H 8309 4205 50  0000 L CNN
-F 2 "" H 8250 4250 50  0001 C CNN
+F 2 "Resistor_SMD:R_0815_2038Metric_Pad1.53x4.00mm_HandSolder" H 8250 4250 50  0001 C CNN
 F 3 "~" H 8250 4250 50  0001 C CNN
 	1    8250 4250
@@
 	8250 3750 8250 4150
 $Comp
-L power:GND #PWR?
+L power:GND #PWR0111
 U 1 1 5E1658A4
 P 6500 4750
-F 0 "#PWR?" H 6500 4500 50  0001 C CNN
+F 0 "#PWR0111" H 6500 4500 50  0001 C CNN
 F 1 "GND" H 6505 4577 50  0000 C CNN
 F 2 "" H 6500 4750 50  0001 C CNN

Commit message: final pcb version
Signed-off-by: Ene Alexandru <ene.alexandru@gmail.com>
Parts:
- removed J10: Conn_01x02, Connector_PinHeader_2.54mm:PinHeader_1x02_P2.54mm_Vertical, symbol Connector_Generic:Conn_01x02
- added J10: Conn_01x03, Connector_PinHeader_2.54mm:PinHeader_1x03_P2.54mm_Vertical, symbol Connector_Generic:Conn_01x03
- R32, R33, R34, R35, R36: footprint Resistor_SMD:R_0815_2038Metric_Pad1.53x4.00mm_HandSolder -> Resistor_SMD:R_0805_2012Metric_Pad1.15x1.40mm_HandSolder
Connections:
- net GND: now also J10.3 (Pin_3)
- net PACK_ALERT: now also U3.14 (PB1); no longer U3.6 (PA0)
- net USART2_RX: now also J10.2 (Pin_2)
- net USART2_TX: now also J10.1 (Pin_1)
Changed lines of the file:
@@
 	-1   0    0    -1
-$EndComp
-$Comp
-L Device:R_Small R33
-U 1 1 5E133DEA
-P 2700 6200
-F 0 "R33" H 2759 6246 50  0000 L CNN
-F 1 "10k" H 2759 6155 50  0000 L CNN
-F 2 "Resistor_SMD:R_0815_2038Metric_Pad1.53x4.00mm_HandSolder" H 2700 6200 50  0001 C CNN
-F 3 "~" H 2700 6200 50  0001 C CNN
-	1    2700 6200
-	1    0    0    -1
 $EndComp
 Wire Wire Line
@@
 F 0 "R32" H 1659 6996 50  0000 L CNN
 F 1 "10k" H 1659 6905 50  0000 L CNN
-F 2 "Resistor_SMD:R_0815_2038Metric_Pad1.53x4.00mm_HandSolder" H 1600 6950 50  0001 C CNN
+F 2 "Resistor_SMD:R_0805_2012Metric_Pad1.15x1.40mm_HandSolder" H 1600 6950 50  0001 C CNN
 F 3 "~" H 1600 6950 50  0001 C CNN
 	1    1600 6950
@@
 Wire Wire Line
 	4950 4650 4950 4750
-Text HLabel 5700 3350 2    50   Input ~ 0
+Text HLabel 4150 4450 0    50   Input ~ 0
 PACK_ALERT
-Wire Wire Line
-	5700 3350 5450 3350
 $Comp
 L bq76920-rescue:ISO7021-bq769xx U?
@@
 	1    0    0    -1
 $EndComp
-$Comp
-L Connector_Generic:Conn_01x02 J10
-U 1 1 5E140FA3
-P 6400 3550
-F 0 "J10" H 6480 3542 50  0000 L CNN
-F 1 "Conn_01x02" H 6480 3451 50  0000 L CNN
-F 2 "Connector_PinHeader_2.54mm:PinHeader_1x02_P2.54mm_Vertical" H 6400 3550 50  0001 C CNN
-F 3 "~" H 6400 3550 50  0001 C CNN
-	1    6400 3550
-	1    0    0    -1
-$EndComp
 Text HLabel 5700 1250 2    50   Input ~ 0
 ISOL_VCC
@@
 Wire Wire Line
 	5450 3550 6200 3550
-Wire Wire Line
-	5450 3650 6200 3650
 Wire Wire Line
 	3100 1350 3800 1350
@@
 F 0 "R34" H 6559 4296 50  0000 L CNN
 F 1 "10k" H 6559 4205 50  0000 L CNN
-F 2 "Resistor_SMD:R_0815_2038Metric_Pad1.53x4.00mm_HandSolder" H 6500 4250 50  0001 C CNN
+F 2 "Resistor_SMD:R_0805_2012Metric_Pad1.15x1.40mm_HandSolder" H 6500 4250 50  0001 C CNN
 F 3 "~" H 6500 4250 50  0001 C CNN
 	1    6500 4250
@@
 F 0 "R35" H 7459 4296 50  0000 L CNN
 F 1 "10k" H 7459 4205 50  0000 L CNN
-F 2 "Resistor_SMD:R_0815_2038Metric_Pad1.53x4.00mm_HandSolder" H 7400 4250 50  0001 C CNN
+F 2 "Resistor_SMD:R_0805_2012Metric_Pad1.15x1.40mm_HandSolder" H 7400 4250 50  0001 C CNN
 F 3 "~" H 7400 4250 50  0001 C CNN
 	1    7400 4250
@@
 F 0 "R36" H 8309 4296 50  0000 L CNN
 F 1 "10k" H 8309 4205 50  0000 L CNN
-F 2 "Resistor_SMD:R_0815_2038Metric_Pad1.53x4.00mm_HandSolder" H 8250 4250 50  0001 C CNN
+F 2 "Resistor_SMD:R_0805_2012Metric_Pad1.15x1.40mm_HandSolder" H 8250 4250 50  0001 C CNN
 F 3 "~" H 8250 4250 50  0001 C CNN
 	1    8250 4250
@@
 Wire Wire Line
 	6500 3950 6500 4150
+Wire Wire Line
+	4150 4450 4450 4450
+$Comp
+L Device:R_Small R33
+U 1 1 5E133DEA
+P 2700 6200
+F 0 "R33" H 2759 6246 50  0000 L CNN
+F 1 "10k" H 2759 6155 50  0000 L CNN
+F 2 "Resistor_SMD:R_0805_2012Metric_Pad1.15x1.40mm_HandSolder" H 2700 6200 50  0001 C CNN
+F 3 "~" H 2700 6200 50  0001 C CNN
+	1    2700 6200
+	1    0    0    -1
+$EndComp
+$Comp
+L Connector_Generic:Conn_01x03 J10
+U 1 1 5E1CDED5
+P 6750 3350
+F 0 "J10" H 6830 3392 50  0000 L CNN
+F 1 "Conn_01x03" H 6830 3301 50  0000 L CNN
+F 2 "Connector_PinHeader_2.54mm:PinHeader_1x03_P2.54mm_Vertical" H 6750 3350 50  0001 C CNN
+F 3 "~" H 6750 3350 50  0001 C CNN
+	1    6750 3350
+	1    0    0    -1
+$EndComp
+$Comp
+L power:GND #PWR?
+U 1 1 5E1CFCD9
+P 6500 3500
+F 0 "#PWR?" H 6500 3250 50  0001 C CNN
+F 1 "GND" H 6505 3327 50  0000 C CNN
+F 2 "" H 6500 3500 50  0001 C CNN
+F 3 "" H 6500 3500 50  0001 C CNN
+	1    6500 3500
+	1    0    0    -1
+$EndComp
+Wire Wire Line
+	6200 3550 6200 3250
+Wire Wire Line
+	6200 3250 6550 3250
+Wire Wire Line
+	6550 3350 6300 3350
+Wire Wire Line
+	6300 3350 6300 3650
+Wire Wire Line
+	5450 3650 6300 3650
+Wire Wire Line
+	6550 3450 6500 3450
+Wire Wire Line
+	6500 3450 6500 3500
 $EndSCHEMATC
