File: hardware/bq76920/bq76920.kicad_pcb (KiCad board)
At the start: 2 copper layers, 60 x 40 mm, 86 parts, among them J1 BAT+, J10 Conn_01x03, J2 Conn_01x06, J3 therm, J4 boot_switch, J5 BAT-, J6 PACK+, J7 PACK-, J8 Conn_01x04, J9 Conn_01x05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

Commit message: create manufacture data, start prototype production
Signed-off-by: Ene Alexandru <ene.alexandru@gmail.com>
Routing:
- net GND: track 12.6 -> 21.3 mm, vias 9 -> 14
- net /balance section/BAL_C5: track 18.8 -> 19.3 mm
- added copper zone on B.Cu, net /BAT+
Changed lines of the file:
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@@
     (thickness 1.6)
     (drawings 21)
-    (tracks 502)
+    (tracks 515)
     (zones 0)
     (modules 86)
@@
       (drillshape 0)
       (scaleselection 1)
-      (outputdirectory "output/"))
+      (outputdirectory "../../production_data/"))
   )
   (net 0 "")
@@
     (tags "capacitor handsolder")
     (attr smd)
-    (fp_text reference C4 (at -2.475 0.2 180) (layer F.SilkS)
+    (fp_text reference C4 (at -2.575 -0.025 180) (layer F.SilkS)
       (effects (font (size 1 1) (thickness 0.15)))
     )
@@
     (tags "resistor handsolder")
     (attr smd)
-    (fp_text reference R7 (at 2.575 -0.1 180) (layer F.SilkS)
+    (fp_text reference R7 (at 2.6 0 180) (layer F.SilkS)
       (effects (font (size 1 1) (thickness 0.15)))
     )
@@
     (tags "resistor handsolder")
     (attr smd)
-    (fp_text reference R8 (at -2.575 0.3 180) (layer F.SilkS)
+    (fp_text reference R8 (at -2.575 0 180) (layer F.SilkS)
       (effects (font (size 1 1) (thickness 0.15)))
     )
@@
     (tags "capacitor handsolder")
     (attr smd)
-    (fp_text reference C16 (at 3.275 0 90) (layer F.SilkS)
+    (fp_text reference C16 (at 3.275 1.05 90) (layer F.SilkS)
       (effects (font (size 1 1) (thickness 0.15)))
     )
@@
     (tags "capacitor handsolder")
     (attr smd)
-    (fp_text reference C18 (at 3.275 0 90) (layer F.SilkS)
+    (fp_text reference C18 (at 3.275 0.4 90) (layer F.SilkS)
       (effects (font (size 1 1) (thickness 0.15)))
     )
@@
   (segment (start 65.8 45.375) (end 68.425 45.375) (width 0.3) (layer F.Cu) (net 2) (status 10))
   (segment (start 68.425 45.375) (end 69.2 44.6) (width 0.3) (layer F.Cu) (net 2))
-  (via (at 53.2 40.55) (size 0.8) (drill 0.4) (layers F.Cu B.Cu) (net 2))
-  (segment (start 53.2 39.15) (end 53.2 40.55) (width 0.3) (layer F.Cu) (net 2) (status 10))
   (via (at 69.6 24.65) (size 0.8) (drill 0.4) (layers F.Cu B.Cu) (net 2))
   (segment (start 69.6 22.85) (end 69.6 24.65) (width 0.3) (layer F.Cu) (net 2))
   (via (at 67.55 30.25) (size 0.8) (drill 0.4) (layers F.Cu B.Cu) (net 2))
   (segment (start 67.575 30.225) (end 67.55 30.25) (width 0.3) (layer F.Cu) (net 2))
+  (segment (start 67.575 28.755) (end 67.575 30.225) (width 0.3) (layer F.Cu) (net 2))
+  (via (at 65.8 32.3) (size 0.8) (drill 0.4) (layers F.Cu B.Cu) (net 2))
+  (segment (start 65.8 34.025) (end 65.8 32.3) (width 0.3) (layer F.Cu) (net 2))
+  (via (at 75.15 40.05) (size 0.8) (drill 0.4) (layers F.Cu B.Cu) (net 2))
+  (segment (start 75.15 41.45) (end 75.15 40.05) (width 0.3) (layer F.Cu) (net 2))
+  (via (at 51.85 39.175) (size 0.8) (drill 0.4) (layers F.Cu B.Cu) (net 2))
+  (segment (start 53.2 39.15) (end 51.875 39.15) (width 0.3) (layer F.Cu) (net 2))
+  (segment (start 51.875 39.15) (end 51.85 39.175) (width 0.3) (layer F.Cu) (net 2))
+  (via (at 56.925 33.325) (size 0.8) (drill 0.4) (layers F.Cu B.Cu) (net 2))
+  (segment (start 57.9 32.7) (end 57.55 32.7) (width 0.3) (layer F.Cu) (net 2))
+  (segment (start 57.55 32.7) (end 56.925 33.325) (width 0.3) (layer F.Cu) (net 2))
+  (via (at 28.075 56.05) (size 0.8) (drill 0.4) (layers F.Cu B.Cu) (net 2))
+  (segment (start 26.6 56.05) (end 28.075 56.05) (width 0.3) (layer F.Cu) (net 2))
+  (via (at 51.25 26.65) (size 0.8) (drill 0.4) (layers F.Cu B.Cu) (net 2))
+  (segment (start 52.725 26.65) (end 51.25 26.65) (width 0.3) (layer B.Cu) (net 2))
   (segment (start 51.525 33.375) (end 53.55 33.375) (width 0.3) (layer F.Cu) (net 3) (status 20))
   (segment (start 51.1 33.8) (end 51.525 33.375) (width 0.3) (layer F.Cu) (net 3))
@@
   (segment (start 32.4 22.5) (end 29.9 25) (width 0.5) (layer F.Cu) (net 8) (status 20))
   (segment (start 52.35 22.5) (end 32.4 22.5) (width 0.5) (layer F.Cu) (net 8) (status 10))
-  (segment (start 24.5 25) (end 29.9 25) (width 5) (layer B.Cu) (net 8) (status 30))
+  (segment (start 29.9 25) (end 24.5 25) (width 5) (layer F.Cu) (net 8))
   (segment (start 47.2 24.375) (end 46.725 23.9) (width 0.3) (layer F.Cu) (net 9))
   (segment (start 47.2 25.05) (end 47.2 24.375) (width 0.3) (layer F.Cu) (net 9) (status 10))
@@
   (segment (start 39.9 24.7) (end 38.65 24.7) (width 0.3) (layer F.Cu) (net 9) (status 20))
   (segment (start 40.7 23.9) (end 39.9 24.7) (width 0.3) (layer F.Cu) (net 9))
-  (segment (start 52.225 28.825) (end 50.9 27.5) (width 0.3) (layer F.Cu) (net 9))
-  (segment (start 50.9 27.5) (end 50.9 25.6) (width 0.3) (layer F.Cu) (net 9))
-  (segment (start 50.9 25.6) (end 50.35 25.05) (width 0.3) (layer F.Cu) (net 9))
-  (segment (start 47.2 25.05) (end 50.35 25.05) (width 0.3) (layer F.Cu) (net 9) (status 10))
-  (segment (start 53.55 28.825) (end 52.225 28.825) (width 0.3) (layer F.Cu) (net 9) (status 10))
+  (segment (start 53.55 28.825) (end 49.55 28.825) (width 0.3) (layer F.Cu) (net 9))
+  (segment (start 49.55 28.825) (end 48.925 28.2) (width 0.3) (layer F.Cu) (net 9))
+  (segment (start 48.925 28.2) (end 48.925 25.4) (width 0.3) (layer F.Cu) (net 9))
+  (segment (start 48.575 25.05) (end 47.2 25.05) (width 0.3) (layer F.Cu) (net 9))
+  (segment (start 48.925 25.4) (end 48.575 25.05) (width 0.3) (layer F.Cu) (net 9))
   (segment (start 45.2 27.1) (end 47.2 27.1) (width 0.3) (layer F.Cu) (net 10) (status 30))
   (segment (start 47.2 27.1) (end 47.2 29.95) (width 0.3) (layer F.Cu) (net 10) (status 30))
@@
     (polygon
       (pts
-        (xy 20 20) (xy 80 20) (xy 80 60) (xy 20 60)
+        (xy 20 28.739063) (xy 33.1 28.750001) (xy 33.1 19.996876) (xy 80 20) (xy 80 60)
+        (xy 20 60)
       )
     )
@@
       )
     )
+  )
+  (zone (net 8) (net_name /BAT+) (layer B.Cu) (hatch edge 0.508)
+    (connect_pads yes (clearance 0.508))
+    (min_thickness 0.254)
+    (fill yes (arc_segments 32) (thermal_gap 0.508) (thermal_bridge_width 0.508))
+    (polygon
+      (pts
+        (xy 32.5 28) (xy 20 28) (xy 20 20) (xy 32.5 20)
+      )
+    )
